File: kicad/actuators/mcu.kicad_sch (KiCad schematic)
At the start: 13 parts, among them J5 Conn_02x03_Odd_Even, U6 STM32G431R6Tx

Commit message: completed the actuator pcb
Parts:
- removed C17, C18, C19, C20, C21, C22: 100nf, Capacitor_SMD:C_0603_1608Metric, symbol Device:C
- removed C23: 1uF, Capacitor_SMD:C_0603_1608Metric, symbol Device:C
- removed C24: 4.7uF, Capacitor_SMD:C_0603_1608Metric, symbol Device:C
- removed C25: C, symbol Device:C
- removed J5: Conn_02x03_Odd_Even, symbol Connector_Generic:Conn_02x03_Odd_Even
- removed R17, R18: 10k, symbol Device:R_US
- removed U6: STM32G431R6Tx, Package_QFP:LQFP-64_10x10mm_P0.5mm, symbol MCU_ST_STM32G4:STM32G431R6Tx
