File: kicad/actuators/wheels.kicad_sch (KiCad schematic)
At the start: 48 parts, among them J1 Conn_01x06, J14 ESTOP SWITCH, J15 LIMIT-SWITCH, J16 LIMIT-SWITCH, J2 Conn_01x06, J3 Conn_01x06, J4 Conn_01x06, U1 DRV8874PWPR, U2 DRV8874PWPR, U3 DRV8874PWPR, U4 DRV8874PWPR, U8 74LVC1G08

Commit message: completed the actuator pcb
Parts:
- C27: renamed from C4; footprint Capacitor_SMD:C_0603_1608Metric -> Capacitor_SMD:CP_Elec_5x5.3
- C28: renamed from C12; footprint Capacitor_SMD:C_0603_1608Metric -> Capacitor_SMD:CP_Elec_5x5.3
- C35: renamed from C8; footprint Capacitor_SMD:C_0603_1608Metric -> Capacitor_SMD:CP_Elec_5x5.3
- C36: renamed from C16; footprint Capacitor_SMD:C_0603_1608Metric -> Capacitor_SMD:CP_Elec_5x5.3
- J13: renamed from J14; footprint (none) -> Connector_PinHeader_2.54mm:PinHeader_1x02_P2.54mm_Vertical
- J16: renamed from J15; footprint (none) -> Connector_PinHeader_2.54mm:PinHeader_1x02_P2.54mm_Vertical
- J17: renamed from J16; footprint (none) -> Connector_PinHeader_2.54mm:PinHeader_1x02_P2.54mm_Vertical
- R12: renamed from R25; footprint (none) -> Resistor_SMD:R_0603_1608Metric
- R17: renamed from R26; footprint (none) -> Resistor_SMD:R_0603_1608Metric
- R22: renamed from R27; footprint (none) -> Resistor_SMD:R_0603_1608Metric
- U6: renamed from U8; footprint (none) -> Package_TO_SOT_SMD:SOT-23-5
- renumbered C32 to C20, C1 to C21, C2 to C22, C9 to C23, C10 to C24, C3 to C25, C11 to C26, C5 to C29, C6 to C30, C13 to C31, C14 to C32, C7 to C33, C15 to C34, J1 to J14, J3 to J15, J2 to J18, J4 to J19, R9 to R10, R10 to R11, R1 to R13, R2 to R14, R11 to R15, R12 to R16, R5 to R18, R6 to R19, R13 to R20, R14 to R21, R7 to R23, R8 to R24, R15 to R25, R16 to R26, R3 to R8, R4 to R9, U1 to U4, U3 to U5, U2 to U7, U4 to U8
Other:
- moved on the sheet: J13, R12
