File: kicad/actuators/actuators.kicad_sch (KiCad schematic)
At the start: 41 parts, among them J10 Conn_01x03, J11 Conn_01x03, J12 Conn_01x03, J13 Conn_01x03, J18 6V_IN, J19 3V3_IN, J5 Conn_02x03_Odd_Even, J6 Conn_01x06, J7 Conn_01x03, J8 Conn_01x03, J9 Conn_01x03, U5 SN65HVD230, U6 STM32G431R6Tx, U7 DRV8874PWPR

Commit message: completed the actuator pcb
Parts:
- removed R18: 10k, symbol Device:R_US
- added J3: Jumper, Connector_PinHeader_2.54mm:PinHeader_1x02_P2.54mm_Vertical, symbol Connector_Generic:Conn_01x02
- added TP1: Boot, TestPoint:TestPoint_Pad_1.5x1.5mm, symbol Connector:TestPoint
- C1: renamed from C25; footprint (none) -> Capacitor_SMD:C_0603_1608Metric
- C19: renamed from C29; footprint Capacitor_SMD:C_0603_1608Metric -> Capacitor_SMD:CP_Elec_5x5.3
- C2: renamed from C33; footprint (none) -> Capacitor_SMD:C_0603_1608Metric
- C3: renamed from C34; footprint (none) -> Capacitor_SMD:C_0603_1608Metric
- C4: renamed from C35; footprint (none) -> Capacitor_SMD:CP_Elec_10x10.5
- C5: renamed from C36; footprint (none) -> Capacitor_SMD:CP_Elec_10x10.5
- J1: renamed from J19; footprint (none) -> Connector_AMASS:AMASS_XT60-M_1x02_P7.20mm_Vertical
- J10: renamed from J11; footprint (none) -> Connector_PinSocket_2.54mm:PinSocket_1x03_P2.54mm_Vertical
- J11: renamed from J13; footprint (none) -> Connector_PinSocket_2.54mm:PinSocket_1x03_P2.54mm_Vertical
- J12: renamed from J7; footprint (none) -> Connector_PinSocket_2.54mm:PinSocket_1x03_P2.54mm_Vertical
- J2: renamed from J18; footprint (none) -> Connector_AMASS:AMASS_XT60-M_1x02_P7.20mm_Vertical
- J4: renamed from J5; footprint (none) -> Connector_PinHeader_2.54mm:PinHeader_2x03_P2.54mm_Vertical
- J6: renamed from J9; footprint (none) -> Connector_PinSocket_2.54mm:PinSocket_1x03_P2.54mm_Vertical
- J7: renamed from J10; footprint (none) -> Connector_PinSocket_2.54mm:PinSocket_1x03_P2.54mm_Vertical
- J8: renamed from J12; footprint (none) -> Connector_PinSocket_2.54mm:PinSocket_1x03_P2.54mm_Vertical
- J9: renamed from J8; footprint (none) -> Connector_PinSocket_2.54mm:PinSocket_1x03_P2.54mm_Vertical
- R1: renamed from R17; footprint (none) -> Resistor_SMD:R_0603_1608Metric
- R6: renamed from R23; footprint (none) -> Resistor_SMD:R_0603_1608Metric
- R7: renamed from R24; footprint (none) -> Resistor_SMD:R_0603_1608Metric
- renumbered C21 to C10, C22 to C11, C23 to C12, C24 to C13, C30 to C14, C31 to C15, C26 to C16, C27 to C17, C28 to C18, C17 to C6, C18 to C7, C19 to C8, C20 to C9, J6 to J5, R19 to R2, R20 to R3, R21 to R4, R22 to R5, U6 to U1, U7 to U2, U5 to U3
Connections:
- net M1_ENA is gone; now on net M5_ENA: U2.3 (nSLEEP)
- net CAN-D: now also U1.62 (PB9)
- net CAN-R: now also J3.2 (Pin_2)
- net E3A: now also U1.59 (PB6); no longer J5.3 (Pin_3)
- net E3B: now also U1.60 (PB7); no longer J5.4 (Pin_4)
- net M1_ADC: now also U1.8 (PC0); no longer R5.1, U2.6 (IPROPI)
- net M1_DIR: now also U1.30 (PB10); no longer U2.2 (PH/IN2)
- net M1_FAULT: now also U1.52 (PC10); no longer R4.2, U2.4 (nFAULT)
- net M1_PWM: now also U1.42 (PA8); no longer U2.1 (EN/IN1)
- net SR1: now also U1.14 (PA2)
- net SR2: now also U1.17 (PA3)
- net SR3: now also U1.18 (PA4)
- net SR4: now also U1.19 (PA5)
- net SR5: now also U1.46 (PA12)
- net SR6: now also U1.51 (PA15)
- net M3_ADC: now reaches U1.10 (PC2)
- net M4_ADC: now reaches U1.11 (PC3)
- net E1A: now reaches U1.12 (PA0)
- net E1B: now reaches U1.13 (PA1)
- net TOPL: now reaches U1.2 (PC13)
- net E2A: now reaches U1.20 (PA6)
- net E2B: now reaches U1.21 (PA7)
- net M5_FAULT: now reaches U1.22 (PC4)
- net M5_FAULT: now also R4.2, U2.4 (nFAULT)
- net M5_ENA: now reaches U1.23 (PC5)
- net E5A: now reaches U1.24 (PB0)
- net E5A: now also J5.3 (Pin_3)
- net E5B: now reaches U1.25 (PB1)
- net E5B: now also J5.4 (Pin_4)
- net M5_DIR: now reaches U1.26 (PB2)
- net M5_DIR: now also U2.2 (PH/IN2)
- net BOML: now reaches U1.3 (PC14)
- net M2_DIR: now reaches U1.33 (PB11)
- net M3_DIR: now reaches U1.34 (PB12)
- net M4_DIR: now reaches U1.35 (PB13)
- net M5_PWM: now reaches U1.36 (PB14)
- net M5_PWM: now also U2.1 (EN/IN1)
- net E4A: now reaches U1.38 (PC6)
- net E4B: now reaches U1.39 (PC7)
- net nSLEEP: now reaches U1.41 (PC9)
- net M2_PWM: now reaches U1.43 (PA9)
- net M3_PWM: now reaches U1.44 (PA10)
- net M4_PWM: now reaches U1.45 (PA11)
- net M2_FAULT: now reaches U1.53 (PC11)
- net M3_FAULT: now reaches U1.54 (PC12)
- net M4_FAULT: now reaches U1.55 (PD2)
- net MOTOR_RUN: now reaches U1.56 (PB3)
- net M5_ADC: now reaches U1.57 (PB4)
- net M5_ADC: now also R5.1, U2.6 (IPROPI)
- net MOTOR_EN: now reaches U1.58 (PB5)
- net at U1.61 (PB8): now also J3.1 (Pin_1), TP1.1
- net M2_ADC: now reaches U1.9 (PC1)
- net M3A renamed M5A
- net M3B renamed M5B
- no-connect marks 1 -> 6
Other:
- sheet Wheels ports: added BOML, E1A, E1B, E2A, E2B, E3A, E3B, E4A, E4B, M1_ADC, M1_DIR, M1_FAULT, M1_PWM, M2_ADC, M2_DIR, M2_FAULT, M2_PWM, M3_ADC, M3_DIR, M3_FAULT, M3_PWM, M4_ADC, M4_DIR, M4_FAULT, M4_PWM, MOTOR_EN, MOTOR_RUN, TOPL, nSLEEP; removed none

Commit message: updated the radio board and changed the servo headers to 6v from 3v3
Connections:
- net +3V3: no longer J10.2 (Pin_2), J11.2 (Pin_2), J6.2 (Pin_2), J7.2 (Pin_2), J8.2 (Pin_2), J9.2 (Pin_2)
- net +6V: now also J10.2 (Pin_2), J11.2 (Pin_2), J6.2 (Pin_2), J7.2 (Pin_2), J8.2 (Pin_2), J9.2 (Pin_2)
Changed lines of the file:
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@@
 	)
 	(symbol
-		(lib_id "power:+3V3")
-		(at 172.72 52.07 0)
-		(unit 1)
-		(body_style 1)
-		(exclude_from_sim no)
-		(in_bom yes)
-		(on_board yes)
-		(in_pos_files yes)
-		(dnp no)
-		(fields_autoplaced yes)
-		(property "Reference" "#PWR028"
-			(at 172.72 55.88 0)
-			(hide yes)
-			(show_name no)
-			(do_not_autoplace no)
-			(effects
-				(font
-					(size 1.27 1.27)
-				)
-			)
-		)
-		(property "Value" "+3V3"
-			(at 172.72 46.99 0)
-			(show_name no)
-			(do_not_autoplace no)
-			(effects
-				(font
-					(size 1.27 1.27)
-				)
-			)
-		)
-		(property "Footprint" ""
-			(at 172.72 52.07 0)
-			(hide yes)
-			(show_name no)
-			(do_not_autoplace no)
-			(effects
-				(font
-					(size 1.27 1.27)
-				)
-			)
-		)
-		(property "Datasheet" ""
-			(at 172.72 52.07 0)
-			(hide yes)
-			(show_name no)
-			(do_not_autoplace no)
-			(effects
-				(font
-					(size 1.27 1.27)
-				)
-			)
-		)
-		(property "Description" "Power symbol creates a global label with name \"+3V3\""
-			(at 172.72 52.07 0)
-			(hide yes)
-			(show_name no)
-			(do_not_autoplace no)
-			(effects
-				(font
-					(size 1.27 1.27)
-				)
-			)
-		)
-		(pin "1"
-		)
-		(instances
-			(project "actuators"
-				(path "/d2c51b21-75fb-4787-ab14-f8a2e4e8f6ca"
-					(reference "#PWR028")
-					(unit 1)
-				)
-			)
-		)
-	)
-	(symbol
 		(lib_id "Connector_Generic:Conn_01x03")
 		(at 160.02 62.23 0)
@@
 					(unit 1)
 				)
+			)
+		)
+	)
+	(symbol
+		(lib_id "power:+6V")
+		(at 172.72 52.07 0)
+		(unit 1)
+		(body_style 1)
+		(exclude_from_sim no)
+		(in_bom yes)
+		(on_board yes)
+		(in_pos_files yes)
+		(dnp no)
+		(fields_autoplaced yes)
+		(property "Reference" "#PWR028"
+			(at 172.72 55.88 0)
+			(hide yes)
+			(show_name no)
+			(do_not_autoplace no)
+			(effects
+				(font
+					(size 1.27 1.27)
+				)
+			)
+		)
+		(property "Value" "+6V"
+			(at 172.72 46.99 0)
+			(show_name no)
+			(do_not_autoplace no)
+			(effects
+				(font
+					(size 1.27 1.27)
+				)
+			)
+		)
+		(property "Footprint" ""
+			(at 172.72 52.07 0)
+			(hide yes)
+			(show_name no)
+			(do_not_autoplace no)
+			(effects
+				(font
+					(size 1.27 1.27)
+				)
+			)
+		)
+		(property "Datasheet" ""
+			(at 172.72 52.07 0)
+			(hide yes)
+			(show_name no)
+			(do_not_autoplace no)
+			(effects
+				(font
+					(size 1.27 1.27)
+				)
+			)
+		)
+		(property "Description" "Power symbol creates a global label with name \"+6V\""
+			(at 172.72 52.07 0)
+			(hide yes)
+			(show_name no)
+			(do_not_autoplace no)
+			(effects
+				(font
+					(size 1.27 1.27)
+				)
+			)
+		)
+		(pin "1"
+		)
+		(instances
+			(project "actuators"
+				(path "/d2c51b21-75fb-4787-ab14-f8a2e4e8f6ca"
+					(reference "#PWR028")
+					(unit 1)
+				)

Commit message: completed the radio board, and making power board
Parts:
- added C37: 100nF, Capacitor_SMD:C_0603_1608Metric, symbol Device:C
- added C38: 470uf, Capacitor_SMD:CP_Elec_10x10.5, symbol Device:C_Polarized
- added J20: 6V2_IN, Connector_AMASS:AMASS_XT30U-M_1x02_P5.0mm_Vertical, symbol Connector_Generic:Conn_01x02
- J1, J2: footprint Connector_AMASS:AMASS_XT60-M_1x02_P7.20mm_Vertical -> Connector_AMASS:AMASS_XT30U-M_1x02_P5.0mm_Vertical
Connections:
- net +6V: no longer J10.2 (Pin_2), J11.2 (Pin_2), J6.2 (Pin_2), J7.2 (Pin_2), J8.2 (Pin_2), J9.2 (Pin_2)
- net GND: now also C37.2, C38.2, J20.2 (Pin_2)
- new net +6V2: C37.1, C38.1, J10.2 (Pin_2), J11.2 (Pin_2), J20.1 (Pin_1), J6.2 (Pin_2), J7.2 (Pin_2), J8.2 (Pin_2), J9.2 (Pin_2)
