File: kicad/main/main.kicad_sch (KiCad schematic)
At the start: 0 parts

Commit message: wrote down the Journal
Parts:
- added BT1: Battery_Cell, symbol Device:Battery_Cell
- added C1, C2, C3, C4: 100nF, symbol Device:C
- added D1: BAT54C, Package_TO_SOT_SMD:SOT-23, symbol Diode:BAT54C
- added J1: Conn_01x04, symbol Connector_Generic:Conn_01x04
- added J2: Conn_01x22, symbol Connector_Generic:Conn_01x22
- added J3: HDMI_A, symbol Connector:HDMI_A
- added J4: USB_A, symbol Connector:USB_A
- added Module1: ComputeModule4, CM4IO:Raspberry-Pi-4-Compute-Module, symbol CM4IO:ComputeModule4-CM4
- added R1: 36k, symbol Device:R_US
- added R2: 120, symbol Device:R_US
- added U1: EMC2301-x-ACZL, Package_SO:MSOP-8_3x3mm_P0.65mm, symbol Driver_Motor:EMC2301-x-ACZL
- added U2: PCF85063ATL, Package_DFN_QFN:DFN-10-1EP_2.6x2.6mm_P0.5mm_EP1.3x2.2mm, symbol Timer_RTC:PCF85063ATL
- added U3: 74LVC1G07, symbol 74xGxx:74LVC1G07
- added U4: SN65HVD230, Package_SO:SOIC-8_3.9x4.9mm_P1.27mm, symbol Interface_CAN_LIN:SN65HVD230
- added U5: MCP2515-xST, Package_SO:TSSOP-20_4.4x6.5mm_P0.65mm, symbol Interface_CAN_LIN:MCP2515-xST
- added Y1: 32.768 kHz, symbol Device:Crystal
- added Y2: 16MHz, symbol Device:Crystal
Connections:
- new net: J1.4 (Pin_4), U1.5 (PWM)
- new net: J1.3 (Pin_3), R1.2, U1.6 (TACH)
- new net: U4.1 (D), U5.1 (TXCAN)
- new net: U4.4 (R), U5.2 (RXCAN)
- new net: U5.8 (OSC2), Y2.2
- new net: U5.9 (OSC1), Y2.1
- new net: R2.1, U4.7 (CANH)
- new net: R2.2, U4.6 (CANL)
- new net: U2.2 (OSCO), Y1.1
- new net: U2.1 (OSCI), Y1.2
- new net: BT1.1 (+), D1.1
- new net: C2.1, D1.3, U2.10 (VDD)
- new net +3.3v: J2.22 (Pin_22)
- new net +3V3: C3.1, C4.1, D1.2, R1.1, U4.3 (VCC), U5.20 (VDD)
- new net +5V: C1.1, J1.2 (Pin_2), U1.3 (VDD)
- new net CAM0_C_N: J2.8 (Pin_8)
- new net CAM0_C_P: J2.9 (Pin_9)
- new net CAM0_D0_N: J2.2 (Pin_2)
- new net CAM0_D0_P: J2.3 (Pin_3)
- new net CAM0_D1_N: J2.5 (Pin_5)
- new net CAM0_D1_P: J2.6 (Pin_6)
- new net CAM_GPIO: J2.17 (Pin_17)
- new net CS: U5.18 (~{CS})
- new net DN: J4.2 (D-)
- new net DP: J4.3 (D+)
- new net GND: BT1.2 (-), C1.2, C2.2, C3.2, C4.2, J1.1 (Pin_1), J2.1 (Pin_1), J2.10 (Pin_10), J2.13 (Pin_13), J2.16 (Pin_16), J2.19 (Pin_19), J2.4 (Pin_4), J2.7 (Pin_7), J3.11 (CKS), J3.17 (GND), J3.2 (D2S), J3.5 (D1S), J3.8 (D0S), J3.SH, J4.4 (GND), J4.SH (Shield), U1.4 (GND), U2.5 (VSS), U4.2 (GND), U4.8 (Rs), U5.10 (VSS)
- new net HDMI0_CEC: J3.13 (CEC)
- new net HDMI0_CK_N: J3.12 (CK-)
- new net HDMI0_CK_P: J3.10 (CK+)
- new net HDMI0_D0_N: J3.9 (D0-)
- new net HDMI0_D0_P: J3.7 (D0+)
- new net HDMI0_D1_N: J3.6 (D1-)
- new net HDMI0_D1_P: J3.4 (D1+)
- new net HDMI0_D2_N: J3.3 (D2-)
- new net HDMI0_D2_P: J3.1 (D2+)
- new net HDMI0_HOTPLUG: J3.19 (HPD)
- new net HDMI0_SCL: J3.15 (SCL)
- new net HDMI0_SDA: J3.16 (SDA)
- new net HDMI_5v: J3.18 (+5V)
- new net INT: U2.4 (~{INT}), U3.2, U5.13 (~{INT})
- new net MISO: U5.17 (SO)
- new net MOSI: U5.16 (SI)
- new net SCK: U5.14 (SCK)
- new net SCL: U1.2 (SMCLK), U2.7 (SCL)
- new net SCL1: J2.20 (Pin_20)
- new net SDA: U1.1 (SMDATA), U2.6 (SDA)
- new net SDA1: J2.21 (Pin_21)
- new net VBUS: J4.1 (VBUS)
- no-connect marks 0 -> 11
Other:
- note added: "Camera"
- note added: "Fan Controller"

Commit message: completed the carrier board schematic
Parts:
- removed C1: 100nF, symbol Device:C
- removed D1: BAT54C, Package_TO_SOT_SMD:SOT-23, symbol Diode:BAT54C
- removed J1: Conn_01x04, symbol Connector_Generic:Conn_01x04
- removed J2: Conn_01x22, symbol Connector_Generic:Conn_01x22
- removed J3: HDMI_A, symbol Connector:HDMI_A
- removed R1: 36k, symbol Device:R_US
- removed U1: EMC2301-x-ACZL, Package_SO:MSOP-8_3x3mm_P0.65mm, symbol Driver_Motor:EMC2301-x-ACZL
- removed U2: PCF85063ATL, Package_DFN_QFN:DFN-10-1EP_2.6x2.6mm_P0.5mm_EP1.3x2.2mm, symbol Timer_RTC:PCF85063ATL
- removed U3: 74LVC1G07, symbol 74xGxx:74LVC1G07
- removed Y1: 32.768 kHz, symbol Device:Crystal
- added C10, C11, C12, C5, C6, C7: 100nF, Capacitor_SMD:C_0603_1608Metric, symbol Device:C
- added C3: 22pF, Capacitor_SMD:C_0603_1608Metric, symbol Device:C
- added C8: 10uF, Capacitor_SMD:C_0805_2012Metric, symbol Device:C
- added C9: 100n, Capacitor_SMD:C_0402_1005Metric, symbol Device:C
- added D1: LED Green, LED_SMD:LED_0805_2012Metric, symbol Device:LED
- added D3: BAT54C-7-F, Package_TO_SOT_SMD:SOT-23, symbol Diode:BAT54C
- added J1: Conn_02x07_Odd_Even, Connector_PinHeader_2.54mm:PinHeader_2x07_P2.54mm_Vertical, symbol Connector_Generic:Conn_02x07_Odd_Even
- added J11: 690-019-298-412, CM4IO:EDAC 690-019-298-412, symbol CM4IO:HDMI_A_1.4
- added J2: Conn_02x04_Odd_Even, Connector_PinHeader_2.54mm:PinHeader_2x04_P2.54mm_Vertical, symbol Connector_Generic:Conn_02x04_Odd_Even
- added J3: Conn_01x06, Connector_Molex:Molex_PicoBlade_53047-0610_1x06_P1.25mm_Vertical, symbol Connector_Generic:Conn_01x06
- added J4: Conn_02x20_Odd_Even, Connector_PinHeader_2.54mm:PinHeader_2x20_P2.54mm_Vertical, symbol Connector_Generic:Conn_02x20_Odd_Even
- added J5: Conn_01x03, Connector:FanPinHeader_1x03_P2.54mm_Vertical, symbol Connector_Generic:Conn_01x03
- added J6: THD-02-R, Connector_PinHeader_2.54mm:PinHeader_2x02_P2.54mm_Vertical, symbol Connector_Generic:Conn_02x02_Odd_Even
- added J7: Conn_01x22_Female, CM4IO:Hirose_FH12-22S-0.5SH_1x22-1MP_P0.50mm_Horizontal, symbol Connector:Conn_01x22_Female
- added J8: Conn_01x04, Connector:FanPinHeader_1x04_P2.54mm_Vertical, symbol Connector_Generic:Conn_01x04
- added J9: Micro_SD_Card_Det, CM4IO:SDCARD_MOLEX_503398-1892, symbol Connector:Micro_SD_Card_Det
- added R1, R2: 10k, Resistor_SMD:R_0603_1608Metric, symbol Device:R
- added R10, R11: 510k, Resistor_SMD:R_0603_1608Metric, symbol Device:R
- added R4: 12k, Resistor_SMD:R_0603_1608Metric, symbol Device:R
- added R5: 36k, Resistor_SMD:R_0603_1608Metric, symbol Device:R_US
- added R6, R7: 470R, Resistor_SMD:R_0603_1608Metric, symbol Device:R
- added R8, R9: R, Resistor_SMD:R_0603_1608Metric, symbol Device:R
- added U1, U10: 74LVC1G07, Package_TO_SOT_SMD:SOT-23-5, symbol 74xGxx:74LVC1G07
- added U11: MagJack-A70-112-331N126, CM4IO:TRJG0926HENL, symbol CM4IO:MagJack-A70-112-331N126
- added U12: PCF85063ATL, Package_DFN_QFN:DFN-10-1EP_2.6x2.6mm_P0.5mm_EP1.3x2.2mm, symbol Timer_RTC:PCF85063ATL
- added U13, U14: TPD4E02B04DQA, Package_SON:USON-10_2.5x1.0mm_P0.5mm, symbol Power_Protection:TPD4E02B04DQA
- added U15: RT9742SNGV, Package_TO_SOT_SMD:SOT-23-3, symbol Power_Management:RT9742SNGV
- added U4: ISM330DHCX, Package_LGA:LGA-14_3x2.5mm_P0.5mm_LayoutBorder3x4y, symbol Sensor_Motion:ISM330DHCX
- added U5: EMC2301-x-ACZL, Package_SO:MSOP-8_3x3mm_P0.65mm, symbol Driver_Motor:EMC2301-x-ACZL
- added U6: RT9742AGJ5F, Package_TO_SOT_SMD:TSOT-23-5, symbol Power_Management:RT9742AGJ5F
- added U7, U8: TPD4EUSB30, Package_SON:USON-10_2.5x1.0mm_P0.5mm, symbol CM4IO:TPD4EUSB30
- added U9: TPD2EUSB30, Package_TO_SOT_SMD:Texas_DRT-3, symbol Power_Protection:TPD2EUSB30
- added Y1: Crystal_GND3, Crystal:Crystal_SMD_3225-4Pin_3.2x2.5mm, symbol Device:Crystal_GND3
- BT1: footprint (none) -> Battery:BatteryHolder_Keystone_3034_1x20mm; Field4 (none) -> Digikey; Field5 (none) -> 36-3034-ND; Field6 (none) -> 3034; Field7 (none) -> Keystone; Part Description (none) -> Battery Retainer Coin, 20.0mm 1 Cell SMD (SMT) Tab
- C1: renamed from C4; footprint (none) -> Capacitor_SMD:C_0603_1608Metric
- C2: value 100nF -> 22pF; footprint (none) -> Capacitor_SMD:C_0603_1608Metric
- C4: renamed from C3; footprint (none) -> Capacitor_SMD:C_0603_1608Metric
- J10: renamed from J4; footprint (none) -> Connector_USB:USB_A_Connfly_DS1095
- R3: renamed from R2; footprint (none) -> Resistor_SMD:R_0603_1608Metric; now not fitted
- Y2: value 16MHz -> 32.768 kHz; footprint (none) -> Crystal:Crystal_SMD_3215-2Pin_3.2x1.5mm
- renumbered U5 to U2, U4 to U3
Connections:
- net CS is gone; now on net GPIO8: U2.18 (~{CS})
- net INT is gone; now on net GPIO25: U2.13 (~{INT})
- net MISO is gone; now on net GPIO9: U2.17 (SO)
- net MOSI is gone; now on net GPIO10: U2.16 (SI)
- net SCK is gone; now on net GPIO11: U2.14 (SCK)
- net +3.3v: now also J7.22 (Pin_22)
- net +3V3: now also Module1.78 (GPIO_VREF(1.8v/3.3v_Input)), C5.1, D1.2 (A), D3.2, J4.1 (Pin_1), J4.17 (Pin_17), R1.1, R10.1, R11.1, R4.1, R5.1, R8.1, U11.15 (LEDG_A), U11.17 (LEDY_A), U4.5 (VDDIO), U4.8 (VDD), U6.5 (VIN)
- net +5V: now also Module1.77 (+5v_(Input)), Module1.79 (+5v_(Input)), Module1.81 (+5v_(Input)), Module1.83 (+5v_(Input)), Module1.85 (+5v_(Input)), Module1.87 (+5v_(Input)), C10.1, C6.1, C7.1, J3.1 (Pin_1), J4.2 (Pin_2), J4.4 (Pin_4), J8.2 (Pin_2), U1.5 (VCC), U10.5 (VCC), U15.1 (VIN), U5.3 (VDD)
- net CAM0_C_N: now also Module1.140 (CAM0_C_N), J7.8 (Pin_8)
- net CAM0_C_P: now also Module1.142 (CAM0_C_P), J7.9 (Pin_9)
- net CAM0_D0_N: now also Module1.128 (CAM0_D0_N), J7.2 (Pin_2)
- net CAM0_D0_P: now also Module1.130 (CAM0_D0_P), J7.3 (Pin_3)
- net CAM0_D1_N: now also Module1.134 (CAM0_D1_N), J7.5 (Pin_5)
- net CAM0_D1_P: now also Module1.136 (CAM0_D1_P), J7.6 (Pin_6)
- net CAM_GPIO: now also Module1.97 (Camera_GPIO), J7.17 (Pin_17)
- net DN: now also Module1.103 (USB2_N), U9.2 (D-)
- net DP: now also Module1.105 (USB2_P), U9.1 (D+)
- net GND: now also Module1.1 (GND), Module1.101 (USB_OTG_ID), Module1.107 (GND), Module1.108 (GND), Module1.113 (GND), Module1.114 (GND), Module1.119 (GND), Module1.120 (GND), Module1.125 (GND), Module1.126 (GND), Module1.13 (GND), Module1.131 (GND), Module1.132 (GND), Module1.137 (GND), Module1.138 (GND), Module1.14 (GND), Module1.144 (GND), Module1.150 (GND), Module1.155 (GND), Module1.156 (GND), Module1.161 (GND), Module1.162 (GND), Module1.167 (GND), Module1.168 (GND), Module1.173 (GND), Module1.174 (GND), Module1.179 (GND), Module1.180 (GND), Module1.185 (GND), Module1.186 (GND), Module1.191 (GND), Module1.192 (GND), Module1.197 (GND), Module1.198 (GND), Module1.2 (GND), Module1.22 (GND), Module1.23 (GND), Module1.32 (GND), Module1.33 (GND), Module1.42 (GND), Module1.43 (GND), Module1.52 (GND), Module1.53 (GND), Module1.59 (GND), Module1.60 (GND), Module1.65 (GND), Module1.66 (GND), Module1.7 (GND), Module1.71 (GND), Module1.74 (GND), Module1.8 (GND), Module1.98 (GND), C10.2, C11.2, C3.2, C5.2, C6.2, C7.2, C8.2, C9.2, J1.1 (Pin_1), J1.10 (Pin_10), J1.12 (Pin_12), J1.3 (Pin_3), J1.7 (Pin_7), J11.11 (CKS), J11.17 (GND), J11.2 (D2S), J11.5 (D1S), J11.8 (D0S), J11.SH1 (SH), J11.SH2 (SH), J11.SH3 (SH), J11.SH4 (SH), J2.2 (Pin_2), J2.4 (Pin_4), J2.6 (Pin_6), J2.8 (Pin_8), J3.4 (Pin_4), J4.14 (Pin_14), J4.20 (Pin_20), J4.25 (Pin_25), J4.30 (Pin_30), J4.34 (Pin_34), J4.39 (Pin_39), J4.6 (Pin_6), J4.9 (Pin_9), J5.3 (Pin_3), J7.1 (Pin_1), J7.10 (Pin_10), J7.13 (Pin_13), J7.16 (Pin_16), J7.19 (Pin_19), J7.4 (Pin_4), J7.7 (Pin_7), J8.1 (Pin_1), J9.11 (SHIELD), J9.6 (VSS), U1.3 (GND), U10.3 (GND), U11.19 (SHIELD), U11.20 (SHIELD), U12.11 (MP), U12.3 (CLKOE), U12.5 (VSS), U13.3 (G), U13.8 (G), U14.3 (G), U14.8 (G), U15.3 (GND), U4.2 (SDx), U4.3 (SCx), U4.6 (GND), U4.7 (GND), U5.4 (GND), U6.2 (GND), U7.3 (GND), U7.8 (GND), U8.3 (GND), U8.8 (GND), U9.3 (GND), Y1.3, Y1.4 (3)
- net HDMI0_CEC: now also Module1.151 (HDMI0_CEC), J11.13 (CEC)
- net HDMI0_CK_N: now also Module1.190 (HDMI0_CLK_N), J11.12 (CK-), U14.5 (IO4)
- net HDMI0_CK_P: now also Module1.188 (HDMI0_CLK_P), J11.10 (CK+), U14.4 (IO3)
- net HDMI0_D0_N: now also Module1.184 (HDMI0_TX0_N), J11.9 (D0-), U14.2 (IO2)
- net HDMI0_D0_P: now also Module1.182 (HDMI0_TX0_P), J11.7 (D0+), U14.1 (IO1)
- net HDMI0_D1_N: now also Module1.178 (HDMI0_TX1_N), J11.6 (D1-), U13.5 (IO4)
- net HDMI0_D1_P: now also Module1.176 (HDMI0_TX1_P), J11.4 (D1+), U13.4 (IO3)
- net HDMI0_D2_N: now also Module1.172 (HDMI0_TX2_N), J11.3 (D2-), U13.2 (IO2)
- net HDMI0_D2_P: now also Module1.170 (HDMI0_TX2_P), J11.1 (D2+), U13.1 (IO1)
- net HDMI0_HOTPLUG: now also Module1.153 (HDMI0_HOTPLUG), J11.19 (HPD/HEAC-)
- net HDMI0_SCL: now also Module1.200 (HDMI0_SCL), J11.15 (SCL)
- net HDMI0_SDA: now also Module1.199 (HDMI0_SDA), J11.16 (SDA)
- net SCL: now also Module1.80 (SCL0), U12.7 (SCL), U4.13 (SCL), U5.2 (SMCLK)
- net SCL1: now also J7.20 (Pin_20)
- net SDA: now also Module1.82 (SDA0), U12.6 (SDA), U4.14 (SDA), U5.1 (SMDATA)
- net SDA1: now also J7.21 (Pin_21)
- net TV_OUT: now reaches Module1.111 (VDAC_COMP)
- net TV_OUT: now also J1.11 (Pin_11)
- net at U2.19 (~{RESET}): now also R1.2
- net at Y2.2: now also U12.1 (OSCI); no longer U2.8 (OSC2)
- net at Y2.1: now also U12.2 (OSCO); no longer U2.9 (OSC1)
- net at R3.1, U3.7 (CANH): now also J5.1 (Pin_1)
- net at R3.2, U3.6 (CANL): now also J5.2 (Pin_2)
- net at BT1.1 (+): now also D3.1
- net TRD0_N: now reaches Module1.10 (Ethernet_Pair0_N)
- net TRD0_N: now also U11.2 (TRD0-), U8.4 (D2+), U8.7
- net TRD2_P: now reaches Module1.11 (Ethernet_Pair2_P)
- net TRD2_P: now also U11.7 (TRD2+), U7.5 (D2-), U7.6
- net TRD0_P: now reaches Module1.12 (Ethernet_Pair0_P)
- net TRD0_P: now also U11.1 (TRD0+), U8.5 (D2-), U8.6
- net ETH_LEDY: now reaches Module1.15 (Ethernet_nLED3(3.3v))
- net ETH_LEDY: now also R7.2
- net SYNC_IN: now reaches Module1.16 (Ethernet_SYNC_IN(1.8v))
- net SYNC_IN: now also J1.8 (Pin_8)
- net ETH_LEDG: now reaches Module1.17 (Ethernet_nLED2(3.3v))
- net ETH_LEDG: now also R6.2
- net SYNC_OUT: now reaches Module1.18 (Ethernet_SYNC_OUT(1.8v))
- net SYNC_OUT: now also J1.9 (Pin_9)
- net EEPROM_nWP: now reaches Module1.20 (EEPROM_nWP)
- net EEPROM_nWP: now also J1.4 (Pin_4)
- net at Module1.21 (PI_nLED_Activity): now also R2.2
- net GPIO26: now reaches Module1.24 (GPIO26)
- net GPIO26: now also J4.37 (Pin_37)
- net GPIO21: now reaches Module1.25 (GPIO21)
- net GPIO21: now also J4.40 (Pin_40)
- net GPIO19: now reaches Module1.26 (GPIO19)
- net GPIO19: now also J4.35 (Pin_35)
- net GPIO20: now reaches Module1.27 (GPIO20)
- net GPIO20: now also J4.38 (Pin_38)
- net GPIO13: now reaches Module1.28 (GPIO13)
- net GPIO13: now also J3.2 (Pin_2), J4.33 (Pin_33)
- net GPIO16: now reaches Module1.29 (GPIO16)
- net GPIO16: now also J4.36 (Pin_36)
- net TRD3_P: now reaches Module1.3 (Ethernet_Pair3_P)
- net TRD3_P: now also U11.9 (TRD3+), U7.1 (D1+), U7.10
- net GPIO6: now reaches Module1.30 (GPIO6)
- net GPIO6: now also J4.31 (Pin_31)
- net GPIO12: now reaches Module1.31 (GPIO12)
- net GPIO12: now also J3.3 (Pin_3), J4.32 (Pin_32)
- net GPIO5: now reaches Module1.34 (GPIO5)
- net GPIO5: now also J4.29 (Pin_29)
- net ID_SC: now reaches Module1.35 (ID_SC)
- net ID_SC: now also J4.28 (Pin_28)
- net ID_SD: now reaches Module1.36 (ID_SD)
- net ID_SD: now also J4.27 (Pin_27)
- net GPIO7: now reaches Module1.37 (GPIO7)
- net GPIO7: now also J4.26 (Pin_26), U4.12 (CS)
- net GPIO11: now reaches Module1.38 (GPIO11)
- net GPIO11: now also J4.23 (Pin_23)
- net GPIO8: now reaches Module1.39 (GPIO8)
- net GPIO8: now also J4.24 (Pin_24)
- net TRD1_P: now reaches Module1.4 (Ethernet_Pair1_P)
- net TRD1_P: now also U11.3 (TRD1+), U8.1 (D1+), U8.10
- net GPIO9: now reaches Module1.40 (GPIO9)
- net GPIO9: now also J4.21 (Pin_21), U4.1 (SDO/SA0)
- net GPIO25: now reaches Module1.41 (GPIO25)
- net GPIO25: now also J4.22 (Pin_22)
- net GPIO10: now reaches Module1.44 (GPIO10)
- net GPIO10: now also J4.19 (Pin_19)
- net GPIO24: now reaches Module1.45 (GPIO24)
- net GPIO24: now also J4.18 (Pin_18), U4.4 (INT1)
- net GPIO22: now reaches Module1.46 (GPIO22)
- net GPIO22: now also J4.15 (Pin_15)
- net GPIO23: now reaches Module1.47 (GPIO23)
- net GPIO23: now also J4.16 (Pin_16), U4.9 (INT2)
- net GPIO27: now reaches Module1.48 (GPIO27)
- net GPIO27: now also J4.13 (Pin_13)
- net GPIO18: now reaches Module1.49 (GPIO18)
- net GPIO18: now also J4.12 (Pin_12)
- net TRD3_N: now reaches Module1.5 (Ethernet_Pair3_N)
- net TRD3_N: now also U11.10 (TRD3-), U7.2 (D1-), U7.9
- net GPIO17: now reaches Module1.50 (GPIO17)
- net GPIO17: now also J4.11 (Pin_11)
- net GPIO15: now reaches Module1.51 (GPIO15)
- net GPIO15: now also J4.10 (Pin_10)
- net GPIO4: now reaches Module1.54 (GPIO4)
- net GPIO4: now also J4.7 (Pin_7)
- net GPIO14: now reaches Module1.55 (GPIO14)
- net GPIO14: now also J4.8 (Pin_8)
- net GPIO3: now reaches Module1.56 (GPIO3)
- net GPIO3: now also J4.5 (Pin_5)
- net SD_CLK: now reaches Module1.57 (SD_CLK)
- net SD_CLK: now also J9.5 (CLK)
- net GPIO2: now reaches Module1.58 (GPIO2)
- net GPIO2: now also J4.3 (Pin_3)
- net TRD1_N: now reaches Module1.6 (Ethernet_Pair1_N)
- net TRD1_N: now also U11.6 (TRD1-), U8.2 (D1-), U8.9
- net SD_DAT3: now reaches Module1.61 (SD_DAT3)
- net SD_DAT3: now also J9.2 (DAT3/CD)
- net SD_CMD: now reaches Module1.62 (SD_CMD)
- net SD_CMD: now also J9.3 (CMD)
- net SD_DAT0: now reaches Module1.63 (SD_DAT0)
- net SD_DAT0: now also J9.7 (DAT0)
- net SD_DAT1: now reaches Module1.67 (SD_DAT1)
- net SD_DAT1: now also J9.8 (DAT1)
- net SD_DAT2: now reaches Module1.69 (SD_DAT2)
- net SD_DAT2: now also J9.1 (DAT2)
- net SD_EN: now reaches Module1.75 (SD_PWR_ON)
- net SD_EN: now also R4.2, U6.4 (EN)
- net SD_DET: now reaches Module1.76 (Reserved)
- net SD_DET: now also R9.1
- net at Module1.89 (WiFi_nDisable): now also J2.1 (Pin_1)
- net TRD2_N: now reaches Module1.9 (Ethernet_Pair2_N)
- net TRD2_N: now also U11.8 (TRD2-), U7.4 (D2+), U7.7
- net at Module1.91 (BT_nDisable): now also J2.3 (Pin_3)
- net RUN_PG: now reaches Module1.92 (RUN_PG)
- net RUN_PG: now also J2.5 (Pin_5), U1.2
- net nRB: now reaches Module1.93 (nRPIBOOT)
- net AIN1: now reaches Module1.94 (AnalogIP0)
- net AIN1: now also J1.6 (Pin_6)
- net nPLED: now reaches Module1.95 (nPI_LED_PWR)
- net AIN0: now reaches Module1.96 (AnalogIP1)
- net AIN0: now also J1.5 (Pin_5)
- net Global_EN: now reaches Module1.99 (Global_EN)
- net Global_EN: now also J2.7 (Pin_7), U10.4
- net at C2.1: now also U2.8 (OSC2), Y1.2
- new net: C12.1, R11.2, U12.4 (~{INT})
- new net: C8.1, J9.4 (VDD), U6.1 (VOUT)
- new net: C11.1, D3.3, U12.10 (VDD)
- new net: J9.9 (DET_B), R9.2
- new net: C3.1, U2.9 (OSC1), Y1.1
- new net: C12.2, R10.2, U10.2
- new net: J8.3 (Pin_3), R5.2, U5.6 (TACH)
- new net: J1.13 (Pin_13), U1.4
- new net: J11.18 (+5V), U15.2 (VOUT)
- new net: R7.1, U11.18 (LEDY_K)
- new net: J8.4 (Pin_4), U5.5 (PWM)
- new net: J9.10 (DET_A), R8.2
- new net: D1.1 (K), R2.1
- new net: R6.1, U11.16 (LEDG_K)
- new net: C9.1, U11.4 (CT), U11.5 (CT)
- new net GLOBAL_EN: J1.14 (Pin_14)
- new net TR0_TAP: J6.3 (Pin_3), U11.11 (VC1)
- new net TR1_TAP: J6.1 (Pin_1), U11.12 (VC2)
- new net TR2_TAP: J6.2 (Pin_2), U11.13 (VC3)
- new net TR3_TAP: J6.4 (Pin_4), U11.14 (VC4)
- new net nRPIBOOT: J1.2 (Pin_2)
- no-connect marks 11 -> 80
Other:
- note added: "40-Pin Header"
- note added: "A button between pins 13-14 can be used to wake up compute module from power down"
- note added: "Benewake TF-LUNA Micro LiDAR Distance Sensor"
- note added: "CAN"
- note added: "EEPROM write protect = Jumper Pins 3-4"
- note added: "Ethernet"
- note added: "Ethernet POE Protection"
- note added: "Force RPIBOOT = Jumper Pins 1-2"
- note added: "IMU"
- note added: "If compute modules is awake RUN_PG will be high so the button doesn't do anything If the compute module is asleep then RUN_PG will be at 0v and so pull global enable low"
- note added: "POE Header"
- note added: "SD card"
- moved on the sheet: C1, C4, J10, Module1A, Module1B, U2, U3

Commit message: layout the pcb
Parts:
- added R12: DNP, Resistor_SMD:R_0603_1608Metric, symbol Device:R
- added R13: 0, Resistor_SMD:R_0603_1608Metric, symbol Device:R
- Y1: value Crystal_GND3 -> 16MHz
Connections:
- net HDMI0_CK_N: now also U14.1 (IO1); no longer U14.5 (IO4)
- net HDMI0_CK_P: now also U14.2 (IO2); no longer U14.4 (IO3)
- net HDMI0_D0_N: now also U14.4 (IO3); no longer U14.2 (IO2)
- net HDMI0_D0_P: now also U14.5 (IO4); no longer U14.1 (IO1)
- net HDMI0_D1_N: now also U13.1 (IO1); no longer U13.5 (IO4)
- net HDMI0_D1_P: now also U13.2 (IO2); no longer U13.4 (IO3)
- net HDMI0_D2_N: now also U13.4 (IO3); no longer U13.2 (IO2)
- net HDMI0_D2_P: now also U13.5 (IO4); no longer U13.1 (IO1)
- net at C2.1, Y1.2: now also R13.2; no longer U2.8 (OSC2)
- net at C3.1, U2.9 (OSC1), Y1.1: now also R12.2
- new net: R12.1, R13.1, U2.8 (OSC2)
Other:
- moved on the sheet: BT1, C2, C3, Y1

Commit message: completed carrier board routing (almost)
Parts:
- added C13: 10uF, Capacitor_SMD:C_0805_2012Metric, symbol Device:C
- added C14: 100nF, Capacitor_SMD:C_0603_1608Metric, symbol Device:C
- added U16: TPS2041B, Package_TO_SOT_SMD:SOT-23-5, symbol Power_Management:TPS2041B
Connections:
- net SCL1 is gone; now on net SCL: J7.20 (Pin_20)
- net SDA1 is gone; now on net SDA: J7.21 (Pin_21)
- net +5V: now also C14.1, U16.5 (IN)
- net GND: now also C13.2, C14.2, U16.2 (GND), U16.4 (~{EN})
- net TRD1_N: now also U8.1 (D1+), U8.10; no longer U8.2 (D1-), U8.9
- net TRD1_P: now also U8.2 (D1-), U8.9; no longer U8.1 (D1+), U8.10
- net TRD3_N: now also U7.1 (D1+), U7.10; no longer U7.2 (D1-), U7.9
- net TRD3_P: now also U7.2 (D1-), U7.9; no longer U7.1 (D1+), U7.10
- net VBUS: now also C13.1, U16.1 (OUT)
- no-connect marks 80 -> 81
Other:
- moved on the sheet: J10, U9

Commit message: completed the main carrier board
Parts:
- added J12: Power Input, Connector_JST:JST_XH_B3B-XH-A_1x03_P2.50mm_Vertical, symbol Connector_Generic:Conn_01x03
Connections:
- net nRPIBOOT is gone; now on net nRB: J1.2 (Pin_2)
- net +3V3: now also J12.3 (Pin_3)
- net +5V: now also J12.1 (Pin_1)
- net GND: now also J12.2 (Pin_2)
