File: kicad/main/main.kicad_pcb (KiCad board)
At the start: 2 copper layers, 55 parts, among them J1 Conn_02x07_Odd_Even, J10 USB_A, J11 690-019-298-412, J2 Conn_02x04_Odd_Even, J3 Conn_01x06, J4 Conn_02x20_Odd_Even, J5 Conn_01x03, J6 THD-02-R, J7 Conn_01x22_Female, J8 Conn_01x04, J9 Micro_SD_Card_Det, U1 74LVC1G07, U10 74LVC1G07, U11 MagJack-A70-112-331N126, U12 PCF85063ATL, U13 TPD4E02B04DQA, U14 TPD4E02B04DQA, U15 RT9742SNGV, U2 MCP2515-xST, U3 SN65HVD230, U4 ISM330DHCX, U5 EMC2301-x-ACZL, U6 RT9742AGJ5F, U7 TPD4EUSB30, U8 TPD4EUSB30, U9 TPD2EUSB30, Y1 Crystal_GND3, Y2 32.768 kHz

Commit message: layout the pcb
Parts:
- added R12: DNP, Resistor_SMD:R_0603_1608Metric, F.Cu at (125.7, 48.6)
- added R13: 0, Resistor_SMD:R_0603_1608Metric, F.Cu at (126.1, 46.1)
- Y1: value Crystal_GND3 -> 16MHz
- moved BT1 690.1 mm to (64.8, 96.2), turned to 90 degrees
- moved D3 689.9 mm to (71.1, 83.4), turned to 90 degrees
- moved C11 674.6 mm to (76.3, 100.7), turned to -90 degrees
- moved C8 671.2 mm to (87.1, 64.2)
- moved U6 670.9 mm to (73.5, 54.8)
- moved C12 670.0 mm to (81.0, 103.6)
- moved J1 666.6 mm to (75.5, 112.1), turned to 90 degrees
- moved C10 665.5 mm to (85.5, 98.4), turned to 180 degrees
- moved J4 657.4 mm to (74.5, 37.3), turned to 90 degrees
- moved U4 638.3 mm to (119.9, 52.2), turned to 90 degrees
- moved U9 635.7 mm to (125.7, 107.4), turned to -90 degrees
- moved J7 633.5 mm to (60.8, 69.3), turned to -90 degrees
- moved U12 632.4 mm to (78.9, 100.8), turned to 90 degrees
- moved R6 631.8 mm to (125.4, 63.7), turned to 180 degrees
- moved R7 631.5 mm to (125.4, 61.7), turned to 180 degrees
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Connections:
- C2 pad 1: Net-(U2-OSC2) -> Net-(C2-Pad1)
- U13 pad 1: /HDMI0_D2_P -> /HDMI0_D1_N
- U13 pad 2: /HDMI0_D2_N -> /HDMI0_D1_P
- U13 pad 4: /HDMI0_D1_P -> /HDMI0_D2_N
- U13 pad 5: /HDMI0_D1_N -> /HDMI0_D2_P
- U14 pad 1: /HDMI0_D0_P -> /HDMI0_CK_N
- U14 pad 2: /HDMI0_D0_N -> /HDMI0_CK_P
- U14 pad 4: /HDMI0_CK_P -> /HDMI0_D0_N
- U14 pad 5: /HDMI0_CK_N -> /HDMI0_D0_P
- Y1 pad 2: Net-(U2-OSC2) -> Net-(C2-Pad1)
Routing:
- net Net-(U2-OSC2): track 0.00 -> 4.39 mm
- net Net-(C2-Pad1): track 0.00 -> 4.13 mm
- net Net-(U2-OSC1): track 0.00 -> 4.02 mm

Commit message: completed carrier board routing (almost)
Parts:
- added C13: 10uF, Capacitor_SMD:C_0805_2012Metric, F.Cu at (130.6, 111.2)
- added C14: 100nF, Capacitor_SMD:C_0603_1608Metric, F.Cu at (129.1, 114.8)
- added U16: TPS2041B, Package_TO_SOT_SMD:SOT-23-5, F.Cu at (127.5, 111.6)
- moved U15 208.5 mm to (69.6, 64.2), turned to -135 degrees
- moved R9 204.3 mm to (64.0, 42.7), turned to 180 degrees
- moved R8 203.4 mm to (63.9, 44.5), turned to 180 degrees
- moved R5 160.2 mm to (102.6, 98.1), turned to -90 degrees
- moved U5 147.4 mm to (106.7, 101.5), turned to 180 degrees
- moved R2 147.1 mm to (119.0, 59.8), turned to 90 degrees
- moved J3 140.5 mm to (122.9, 113.7), turned to 180 degrees
- moved C5 138.7 mm to (122.3, 53.8), turned to -90 degrees
- moved C7 134.9 mm to (111.1, 100.5), turned to 90 degrees
- moved C6 124.7 mm to (121.1, 110.7), turned to 180 degrees
- moved D1 123.8 mm to (121.0, 59.8), turned to 90 degrees
- moved J1 68.4 mm to (142.0, 96.0), turned to 180 degrees
- moved J11 68.3 mm to (64.2, 69.3), turned to -90 degrees
- moved U14 59.1 mm to (69.2, 69.1), turned to 0 degrees
- moved U13 57.1 mm to (69.2, 72.5), turned to 0 degrees
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Connections:
- J7 pad 20: /SCL1 -> /SCL
- J7 pad 21: /SDA1 -> /SDA
- U7 pad 1: /TRD3_P -> /TRD3_N
- U7 pad 10: /TRD3_P -> /TRD3_N
- U7 pad 2: /TRD3_N -> /TRD3_P
- U7 pad 9: /TRD3_N -> /TRD3_P
- U8 pad 1: /TRD1_P -> /TRD1_N
- U8 pad 10: /TRD1_P -> /TRD1_N
- U8 pad 2: /TRD1_N -> /TRD1_P
- U8 pad 9: /TRD1_N -> /TRD1_P
Routing:
- net +3V3: track 0.00 -> 299.7 mm, vias 0 -> 6
- net +5V: track 0.00 -> 249.3 mm, vias 0 -> 4
- net /SCL: track 0.00 -> 169.9 mm, vias 0 -> 5
- net /SDA: track 0.00 -> 163.6 mm, vias 0 -> 5
- net GND: track 0.00 -> 156.9 mm, vias 0 -> 2426
- net /CAM_GPIO: track 0.00 -> 94.8 mm
- net /GPIO13: track 0.00 -> 90.8 mm, vias 0 -> 2
- net /GPIO12: track 0.00 -> 89.9 mm, vias 0 -> 2
- net /GPIO9: track 0.00 -> 86.3 mm, vias 0 -> 2
- net /RUN_PG: track 0.00 -> 79.5 mm, vias 0 -> 2
- net /GPIO15: track 0.00 -> 79.4 mm, vias 0 -> 1
- net /GPIO11: track 0.00 -> 79.1 mm, vias 0 -> 2
- net /GPIO8: track 0.00 -> 79.0 mm
- net /SD_DAT1: track 0.00 -> 71.9 mm
- net /SD_DAT0: track 0.00 -> 70.3 mm
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- added copper zone on B.Cu, net GND
- added copper zone on F.Cu, net GND
- added copper zone on In1.Cu, net GND
- added copper zone on In2.Cu, net GND
- added copper zone on In3.Cu, net GND
- added copper zone on In4.Cu, net GND
Other:
- board outline added: 88.5 x 84.7 mm
- copper layers 2 -> 6

Commit message: completed the main carrier board
Parts:
- added J12: Power Input, Connector_JST:JST_XH_B3B-XH-A_1x03_P2.50mm_Vertical, F.Cu at (67.0, 36.9)
- moved D1 4.36 mm to (125.3, 59.2), turned to 0 degrees
- moved R2 4.06 mm to (122.8, 61.4), turned to -90 degrees
- moved U4 2.97 mm to (119.2, 49.3)
- moved C5 2.88 mm to (121.7, 51.0)
- moved C6 1.96 mm to (123.0, 110.2), turned to 90 degrees
- moved U15 0.50 mm to (69.2, 63.9)
- moved D3 0.37 mm to (82.3, 111.0)
- moved U14 0.06 mm to (69.1, 69.1)
Connections:
- J1 pad 2: /nRPIBOOT -> /nRB
Routing:
- net GND: track 156.9 -> 233.9 mm, vias 2426 -> 2071
- net /nRB: track 0.00 -> 71.7 mm, vias 0 -> 1
- net +3V3: track 299.7 -> 347.7 mm, vias 6 -> 8
- net /SDA: track 163.6 -> 195.3 mm, vias 5 -> 3
- net /SCL: track 169.9 -> 201.4 mm
- net /GPIO19: track 39.3 -> 65.8 mm, vias 1 -> 2
- net /GPIO10: track 66.4 -> 92.3 mm, vias 3 -> 2
- net /CAM_GPIO: track 94.8 -> 70.0 mm, vias 0 -> 2
- net Net-(Module1A-PI_nLED_Activity): track 37.1 -> 15.0 mm
- net /GPIO23: track 65.8 -> 86.7 mm, vias 2 -> 1
- net /ID_SC: track 69.7 -> 49.2 mm
- net +5V: track 249.3 -> 269.2 mm, vias 4 -> 7
- net /GPIO8: track 79.0 -> 59.6 mm, vias 0 -> 1
- net /GPIO13: track 90.8 -> 109.3 mm, vias 2 -> 1
- net /TV_OUT: track 64.0 -> 81.7 mm, vias 1 -> 0
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
Commit message: started work on the radio board
Parts:
- added REF**: MountingHole_3.2mm_M3_DIN965_Pad_TopBottom, MountingHole:MountingHole_3.2mm_M3_DIN965_Pad_TopBottom, F.Cu at (74.1, 89.2)
- added REF**: MountingHole_3.2mm_M3_DIN965_Pad_TopBottom, MountingHole:MountingHole_3.2mm_M3_DIN965_Pad_TopBottom, F.Cu at (140.1, 35.9)
- added REF**: MountingHole_3.2mm_M3_DIN965_Pad_TopBottom, MountingHole:MountingHole_3.2mm_M3_DIN965_Pad_TopBottom, F.Cu at (126.3, 100.2)
Routing:
- net GND: vias 2071 -> 2394
