File: kicad/radio/radio.kicad_pcb (KiCad board)
At the start: 2 copper layers, 15 parts, among them IC1 E22-900M22S, J4 Conn_02x20_Odd_Even, J6 Conn_Coaxial, J8 Conn_Coaxial, Q3 NPN, U9 SIM7080G

Commit message: updated the radio board and changed the servo headers to 6v from 3v3
Parts:
- added C22: 22uF, Capacitor_SMD:C_0805_2012Metric_Pad1.18x1.45mm_HandSolder, F.Cu at (131.6, 132.7)
- added C23: 100nF, Capacitor_SMD:C_0805_2012Metric_Pad1.18x1.45mm_HandSolder, F.Cu at (131.6, 135.7)
- added C24: 100nF, Capacitor_SMD:C_0805_2012Metric_Pad1.18x1.45mm_HandSolder, F.Cu at (131.6, 138.8)
- added C25: 22uF, Capacitor_SMD:C_0805_2012Metric_Pad1.18x1.45mm_HandSolder, F.Cu at (131.6, 141.8)
- added C26: 100nF, Capacitor_SMD:C_0805_2012Metric_Pad1.18x1.45mm_HandSolder, F.Cu at (131.6, 144.8)
- added C27: 100nF, Capacitor_SMD:C_0805_2012Metric_Pad1.18x1.45mm_HandSolder, F.Cu at (131.6, 147.8)
- added C28: 100nF, Capacitor_SMD:C_0805_2012Metric_Pad1.18x1.45mm_HandSolder, F.Cu at (131.6, 150.8)
- added C29: 10uF, Capacitor_SMD:C_0805_2012Metric_Pad1.18x1.45mm_HandSolder, F.Cu at (131.6, 153.8)
- added D2: SS34, Diode_SMD:D_SMA, F.Cu at (138.1, 145.7)
- added J9: Conn_Coaxial, Connector_Coaxial:SMA_Amphenol_132289_EdgeMount, F.Cu at (138.3, 137.3)
- added R21: 53.6k, Resistor_SMD:R_0805_2012Metric_Pad1.20x1.40mm_HandSolder, F.Cu at (121.1, 122.4)
- added R22: 10k, Resistor_SMD:R_0805_2012Metric_Pad1.20x1.40mm_HandSolder, F.Cu at (121.1, 125.4)
- added U1: MT3608, Package_TO_SOT_SMD:SOT-23-6, F.Cu at (144.7, 145.8)
- added U2: TPD4E05U06DQA, Package_SON:USON-10_2.5x1.0mm_P0.5mm, F.Cu at (148.8, 145.7)
- added U7: TXS0102DCT, Package_SO:SSOP-8_2.95x2.8mm_P0.65mm, F.Cu at (137.3, 150.3)
Connections:
- IC1 pad 13: unconnected-(IC1-DIO1-Pad13) -> /DIO1
- IC1 pad 14: unconnected-(IC1-BUSY-Pad14) -> /BUSY
- IC1 pad 15: unconnected-(IC1-NRST-Pad15) -> /GPIO5
- IC1 pad 16: unconnected-(IC1-MISO-Pad16) -> /GPIO9
- IC1 pad 17: unconnected-(IC1-MOSI-Pad17) -> /GPIO10
- IC1 pad 18: unconnected-(IC1-SCK-Pad18) -> /GPIO11
- IC1 pad 19: unconnected-(IC1-NSS-Pad19) -> /GPIO4
- IC1 pad 21: unconnected-(IC1-ANT-Pad21) -> /RF
- IC1 pad 6: unconnected-(IC1-RXEN-Pad6) -> /GPIO17
- IC1 pad 7: unconnected-(IC1-TXEN-Pad7) -> /TXEN
- IC1 pad 8: unconnected-(IC1-DIO2-Pad8) -> /TXEN
- IC1 pad 9: unconnected-(IC1-VCC-Pad9) -> +3V3
- J4 pad 31: /GPIO6 -> /BUSY
- J4 pad 36: /GPIO16 -> /DIO1
- R17 pad 2: /IO45 -> /GPIO18

Commit message: completed the radio board, and making power board
Parts:
- added J2: Conn_01x04, Connector_JST:JST_XH_B4B-XH-A_1x04_P2.50mm_Vertical, F.Cu at (141.7, 120.5)
- added L1: 10uH, Inductor_SMD:L_7.3x7.3_H4.5, F.Cu at (116.9, 74.4)
- added R23: 10k, Resistor_SMD:R_0805_2012Metric_Pad1.20x1.40mm_HandSolder, F.Cu at (138.1, 114.9)
- added R24: 22, Resistor_SMD:R_0805_2012Metric_Pad1.20x1.40mm_HandSolder, B.Cu at (132.1, 99.9)
- added R25: 22, Resistor_SMD:R_0805_2012Metric_Pad1.20x1.40mm_HandSolder, B.Cu at (129.9, 99.9)
- added R26: 22, Resistor_SMD:R_0805_2012Metric_Pad1.20x1.40mm_HandSolder, B.Cu at (134.1, 99.9)
- added R27: 10k, Resistor_SMD:R_0805_2012Metric_Pad1.20x1.40mm_HandSolder, F.Cu at (141.9, 114.9)
- added R28: 10k, Resistor_SMD:R_0805_2012Metric_Pad1.20x1.40mm_HandSolder, F.Cu at (134.2, 114.9)
- added REF**: MountingHole_2.2mm_M2_DIN965_Pad_TopBottom, MountingHole:MountingHole_2.2mm_M2_DIN965_Pad_TopBottom, F.Cu at (112.9, 121.7)
- added REF**: MountingHole_2.2mm_M2_DIN965_Pad_TopBottom, MountingHole:MountingHole_2.2mm_M2_DIN965_Pad_TopBottom, F.Cu at (110.2, 76.2)
- added REF**: MountingHole_2.2mm_M2_DIN965_Pad_TopBottom, MountingHole:MountingHole_2.2mm_M2_DIN965_Pad_TopBottom, F.Cu at (145.0, 110.0)
- added REF**: MountingHole_2.2mm_M2_DIN965_Pad_TopBottom, MountingHole:MountingHole_2.2mm_M2_DIN965_Pad_TopBottom, F.Cu at (146.1, 72.8)
- Card1, R18, U2: moved to B.Cu
- moved U1 70.9 mm to (115.3, 81.3), turned to -90 degrees
- moved D2 66.5 mm to (119.4, 81.9), turned to 90 degrees
- moved U7 61.1 mm to (114.4, 93.7)
- moved IC1 57.9 mm to (122.4, 109.4), turned to 180 degrees
- moved C27 57.1 mm to (118.2, 92.3), turned to 90 degrees
- moved C26 55.4 mm to (110.5, 93.6), turned to 90 degrees
- moved C25 53.8 mm to (120.5, 89.1)
- moved C24 52.9 mm to (120.5, 87.0)
- moved C23 52.2 mm to (114.3, 86.6), turned to 180 degrees
- moved C22 51.3 mm to (114.3, 84.5), turned to 180 degrees
- moved R17 49.8 mm to (110.1, 85.5), turned to 180 degrees
- moved U2 46.9 mm to (122.4, 106.9), turned to 90 degrees
- moved R22 45.2 mm to (112.4, 81.0), turned to -90 degrees
- moved C29 42.9 mm to (110.6, 116.4), turned to -90 degrees
- moved R21 42.7 mm to (110.3, 81.1), turned to 90 degrees
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Connections:
- IC1 pad 21: /RF -> /RF-3
- J4 pad 15: /GPIO22 -> /ALERT
- J9 pad 1: /RF -> /RF-3
- U2 pad 1: /SIM_CLK -> /SIM_VDD
- U2 pad 2: /SIM_DATA -> /SIM_RST
- U2 pad 4: /SIM_VDD -> /SIM_CLK
- U2 pad 5: /SIM_RST -> /SIM_DATA
- U9 pad 15: /SIM_DATA -> Net-(U9-SIM_DATA)
- U9 pad 16: /SIM_CLK -> Net-(U9-SIM_CLK)
- U9 pad 17: /SIM_RST -> Net-(U9-SIM_RST)
Routing:
- net +3V3: track 0.00 -> 183.2 mm, vias 0 -> 1
- net /GPIO2: track 0.00 -> 66.9 mm
- net /GPIO3: track 0.00 -> 64.3 mm
- net /ALERT: track 0.00 -> 56.1 mm
- net +3V8: track 0.00 -> 55.3 mm, vias 0 -> 3
- net /GPIO5: track 0.00 -> 52.2 mm
- net /BUSY: track 0.00 -> 43.7 mm
- net /GPIO4: track 0.00 -> 43.5 mm, vias 0 -> 1
- net /VDD_EXT: track 0.00 -> 41.6 mm, vias 0 -> 2
- net /NETLIGHT: track 0.00 -> 37.7 mm, vias 0 -> 2
- net /STATUS: track 0.00 -> 37.0 mm, vias 0 -> 2
- net GND: track 0.00 -> 33.5 mm, vias 0 -> 761
- net /GPIO17: track 0.00 -> 32.3 mm, vias 0 -> 1
- net /GPIO10: track 0.00 -> 30.9 mm, vias 0 -> 1
- net /GPIO9: track 0.00 -> 29.3 mm, vias 0 -> 1
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- added copper zone on B.Cu, net GND
- added copper zone on F.Cu, net GND
- added copper zone on In1.Cu, net GND
- added copper zone on In2.Cu, net GND
Other:
- board outline added: 48.6 x 54.5 mm
- copper layers 2 -> 4
