File: kicad/radio/radio.kicad_sch (KiCad schematic)
At the start: 31 parts, among them IC1 E22-900M22S, J4 Conn_02x20_Odd_Even, J6 Conn_Coaxial, J8 Conn_Coaxial, J9 Conn_Coaxial, Q3 NPN, U1 MT3608, U2 TPD4E05U06DQA, U7 TXS0102DCT, U9 SIM7080G

Commit message: updated the radio board and changed the servo headers to 6v from 3v3
Parts:
- removed R1: 53.6k, symbol Device:R
- removed R2: 10k, symbol Device:R
- added R21: 53.6k, Resistor_SMD:R_0805_2012Metric_Pad1.20x1.40mm_HandSolder, symbol Device:R
- added R22: 10k, Resistor_SMD:R_0805_2012Metric_Pad1.20x1.40mm_HandSolder, symbol Device:R
- added R24, R25, R26: 22, Resistor_SMD:R_0805_2012Metric_Pad1.20x1.40mm_HandSolder, symbol Device:R
- L1: footprint (none) -> Inductor_SMD:L_7.3x7.3_H4.5
Connections:
- net GPIO16 is gone; now on net DIO1: J4.36 (Pin_36)
- net GPIO6 is gone; now on net BUSY: J4.31 (Pin_31)
- net IO45 is gone; now on net GPIO18: R17.2
- net MISO is gone; now on net GPIO9: IC1.16 (MISO)
- net MOSI is gone; now on net GPIO10: IC1.17 (MOSI)
- net NRST is gone; now on net GPIO5: IC1.15 (NRST)
- net NSS is gone; now on net GPIO4: IC1.19 (NSS)
- net RXD is gone; now on net GPIO15: U7.8 (B1)
- net RXEN is gone; now on net GPIO17: IC1.6 (RXEN)
- net SCK is gone; now on net GPIO11: IC1.18 (SCK)
- net TXD is gone; now on net GPIO14: U7.1 (B2)
- net +3V8: now also R21.1
- net GND: now also R22.2
- net SIM_CLK: now also R24.1; no longer U9.16 (SIM_CLK)
- net SIM_DATA: now also R25.1; no longer U9.15 (SIM_DATA)
- net SIM_RST: now also R26.1; no longer U9.17 (SIM_RST)
- net TXEN: now also IC1.8 (DIO2)
- net at U1.3 (FB): now also R21.2, R22.1
- new net: R24.2, U9.16 (SIM_CLK)
- new net: R25.2, U9.15 (SIM_DATA)
- new net: R26.2, U9.17 (SIM_RST)
- no-connect marks 33 -> 32

Commit message: completed the radio board, and making power board
Parts:
- added J2: Conn_01x04, Connector_JST:JST_XH_B4B-XH-A_1x04_P2.50mm_Vertical, symbol Connector_Generic:Conn_01x04
- added R23, R27, R28: 10k, Resistor_SMD:R_0805_2012Metric_Pad1.20x1.40mm_HandSolder, symbol Device:R
Connections:
- net +3V3: now also R23.1, R27.1, R28.1
- net GND: now also J2.4 (Pin_4)
- net GPIO2: now also J2.1 (Pin_1), R27.2
- net GPIO3: now also J2.2 (Pin_2), R23.2
- net RF: no longer IC1.21 (ANT), J9.1 (In)
- net SIM_CLK: now also U2.4 (D2+); no longer U2.1 (D1+)
- net SIM_DATA: now also U2.5 (D2-); no longer U2.2 (D1-)
- net SIM_RST: now also U2.2 (D1-); no longer U2.5 (D2-)
- net SIM_VDD: now also U2.1 (D1+); no longer U2.4 (D2+)
- net GPIO22 renamed ALERT
- net ALERT: now also J2.3 (Pin_3), R28.2
- new net RF-3: IC1.21 (ANT), J9.1 (In)
