File: kicad/power/power/power.kicad_sch (KiCad schematic)
At the start: 0 parts

Commit message: completed the buck section
Parts:
- added C1, C10, C11, C12, C2, C3, C4, C5, C6, C7, C8, C9: C, symbol Device:C
- added L1, L2, L3: L, symbol Device:L
- added U1, U2, U3: LMR33640ADDA, Package_SO:Texas_HSOP-8-1EP_3.9x4.9mm_P1.27mm_ThermalVias, symbol Regulator_Switching:LMR33640ADDA
Connections:
- new net: C6.1, U2.6 (VCC)
- new net: L3.1, U3.5 (FB)
- new net: C1.1, U1.7 (BOOT)
- new net: C1.2, U1.8 (SW)
- new net: L1.1, U1.5 (FB)
- new net: C4.1, U1.6 (VCC)
- new net: C11.1, U3.7 (BOOT)
- new net: C11.2, U3.8 (SW)
- new net: L2.1, U2.5 (FB)
- new net: C7.1, U2.7 (BOOT)
- new net: C7.2, U2.8 (SW)
- new net: C10.1, U3.6 (VCC)
- new net GND: C10.2, C12.2, C2.2, C3.2, C4.2, C5.2, C6.2, C8.2, C9.2, U1.1 (GND), U1.9 (GND), U2.1 (GND), U2.9 (GND), U3.1 (GND), U3.9 (GND)
- new net VIN: C3.1, C5.1, C9.1, U1.2 (VIN), U1.3 (EN), U2.2 (VIN), U2.3 (EN), U3.2 (VIN), U3.3 (EN)
- new net VOUT: C12.1, C2.1, C8.1, L1.2, L2.2, L3.2
- no-connect marks 0 -> 3
Other:
- added sheet 19V bucks (19vbuck.kicad_sch)
